File: design/pcb/63/keycult63.kicad_pcb (KiCad board)
At the start: 4 copper layers, 285 x 94.6 mm, 175 parts, among them SW1 r0c0 Esc, SW10 r0c9 6, SW11 r0c10 7, SW12 r0c11 8, SW13 r0c12 9, SW14 r0c13 0, SW15 r0c14 Bksp, SW16 r1c0 Tab, SW17 r1c1 Q, SW18 r1c2 W, SW19 r1c3 E, SW2 r0c1 1, SW20 r1c4 R, SW21 r1c5 T, SW22 r1c9 Y, SW23 r1c10 U, SW24 r1c11 I, SW25 r1c12 O, SW26 r1c13 P, SW27 r1c14 \, SW28 r2c0 Caps, SW29 r2c1 A, SW3 r0c2 2, SW30 r2c2 S, SW31 r2c3 D, SW32 r2c4 F, SW33 r2c5 G, SW34 r2c9 H, SW35 r2c10 J, SW36 r2c11 K, SW37 r2c12 L, SW38 r2c13 ;, SW39 r2c14 Enter, SW4 r0c3 3, SW40 r3c0 Shift, SW41 r3c1 Z, SW42 r3c2 X, SW43 r3c3 C, SW44 r3c4 V, SW45 r3c5 B, SW46 r3c9 N, SW47 r3c10 M, SW48 r3c11 ,, SW49 r3c12 ., SW5 r0c4 4, SW50 r3c13 /, SW51 r3c14 Shift, SW52 r4c0 Ctrl, SW53 r4c1 GUI, SW54 r4c2 Alt, SW55 r4c3 Fn, SW56 r4c4 Space, SW57 r4c5 Del, SW58 r4c6 M1, SW59 r4c7 M3, SW6 r0c5 5, SW60 r4c8 M2, SW61 r4c9 Bksp, SW62 r4c10 Space, SW63 r4c11 Fn, SW64 r4c12 Left, SW65 r4c13 Down, SW66 r4c14 Right, SW67 BOOTSEL, SW68 RESET, U1 RP2040, U2 W25Q16JVSSIQ, U3 AP2112K-3.3TRG1, Y1 ABM8-272-T3 12MHz CL10pF

Commit message: feat(pcb): add UDB interface and record paused design checkpoint
Parts:
- added J1: USB / UDB JST-SH, Connector_JST:JST_SH_SM04B-SRSS-TB_1x04-1MP_P1.00mm_Horizontal, B.Cu at (40.6, 112.0)
- TP1: value VBUS_USB / USB LOGICAL -> VBUS_USB / USB TEST
- TP2: value GND / USB LOGICAL -> GND / USB TEST
- TP3: value USB_DM / USB LOGICAL -> USB_DM / USB TEST
- TP4: value USB_DP / USB LOGICAL -> USB_DP / USB TEST
Routing:
- net USB_DP: track 16.8 -> 160.0 mm, vias 2 -> 4
- net USB_DM: track 15.0 -> 156.4 mm, vias 2 -> 4
- net VBUS_USB: track 15.2 -> 109.7 mm, vias 0 -> 2
- net GND: track 24.0 -> 27.3 mm, vias 30 -> 33
Other:
- board text added: "DRAFT C / 63 KEYS - NOT FOR FABRICATION"
- board text added: "J1 UDB: 1 VBUS / 2 D- / 3 D+ / 4 GND; CABLE FIT TBD"
- board text removed: "DRAFT B / 63 KEYS - NOT FOR FABRICATION"
- board text removed: "USB LOGICAL PADS - PINOUT TBD"

Commit message: feat(pcb): adopt external C5-JSH daughterboard assumption
Parts:
- J1: value USB / UDB JST-SH -> USB / C5-JSH JST-SH
Other:
- board text added: "DRAFT D / 63 KEYS - NOT FOR FABRICATION"
- board text added: "J1 TO EXTERNAL C5-JSH: 1 POWER / 2 D- / 3 D+ / 4 GND; F1 RETAINED"
- board text removed: "DRAFT C / 63 KEYS - NOT FOR FABRICATION"
- board text removed: "J1 UDB: 1 VBUS / 2 D- / 3 D+ / 4 GND; CABLE FIT TBD"

Commit message: feat(pcb): reroute USB over the ground reference
Apply the candidate 7628 stackup and 0.29/0.20mm F.Cu pair to both variants. Add local ground stitching and preserve the existing power, matrix and MCU-side copper.

Validate refilled reference coverage, strict ERC/DRC and saved-route replay. Refresh native exports and document the remaining impedance and hardware limits.
Routing:
- net USB_DM: track 156.4 -> 151.4 mm
- net USB_DP: track 160.0 -> 157.4 mm
- net GND: vias 33 -> 36
- added copper zone on B.Cu, net GND
Other:
- board text added: "DRAFT E / 63 KEYS - NOT FOR FABRICATION"
- board text added: "USB F.Cu 0.29/0.20mm; 7628 STACKUP STUDY / IMPEDANCE NOT QUALIFIED"
- board text removed: "DRAFT D / 63 KEYS - NOT FOR FABRICATION"
- board text removed: "J1 TO EXTERNAL C5-JSH: 1 POWER / 2 D- / 3 D+ / 4 GND; F1 RETAINED"

Commit message: feat(pcb): use two 1.5u trackball buttons in both layouts
Parts:
- removed D59: 1N4148W, Diode_SMD:D_SOD-123
- removed SW59: r4c7 M3, Button_Switch_Keyboard:SW_Cherry_MX_1.00u_PCB
- SW58, SW60: footprint Button_Switch_Keyboard:SW_Cherry_MX_1.00u_PCB -> Button_Switch_Keyboard:SW_Cherry_MX_1.50u_PCB
- moved D58 4.76 mm to (161.7, 144.7)
- moved D60 4.76 mm to (190.3, 144.7)
- moved SW60 4.76 mm to (196.8, 133.0)
- moved SW58 4.76 mm to (168.3, 133.0)
Connections:
- U1 pad 27: COL7 -> unconnected-(U1-GPIO16-Pad27)
Routing:
- net COL7: track 163.1 -> 0.00 mm, vias 4 -> 0
- net ROW4: track 359.8 -> 383.1 mm, vias 16 -> 15
- net COL8: track 178.6 -> 165.1 mm
- net K_r4c7: track 10.6 -> 0.00 mm
- net COL6: track 150.5 -> 156.6 mm
- net QSPI_SD2: track 15.9 -> 12.6 mm
- net COL11: track 348.3 -> 348.9 mm
- net K_r4c8: track 10.6 -> 10.7 mm, vias 0 -> 1
- net K_r4c6: vias 0 -> 1
Other:
- board text added: "DRAFT E / 62 KEYS - NOT FOR FABRICATION"
- board text removed: "DRAFT E / 63 KEYS - NOT FOR FABRICATION"
- board text removed: "r4c7"
